File: nrf52_sensor_array.sch (KiCad schematic (older format))
At the start: 73 parts, among them IC1 ADS1299, P1 CONN_2, P2 CONN_2, P3 CONN_01X08, U1 TPS2294x, U2 TPS61222, U3 NRF528XX-QFAA, U4 MPU-9250, U5 INA828, U6 INA828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

Commit message: Remove extraneous stuff from schematic.
Parts:
- removed C10: 10uF, Capacitors_SMD:C_0603, symbol C
- removed C11, C18, C20, C31, C32, C7, C9: 0.1uF, Capacitors_SMD:C_0402, symbol C
- removed C12, C14, C16, C17, C19, C37, C40, C5, C6, C8: 1uF, Capacitors_SMD:C_0402, symbol C
- removed C15: 100µF, Capacitors_SMD:C_0603, symbol CP1
- removed C35, C36: 100nF, Capacitors_SMD:C_0402, symbol C
- removed C4: 1.0nF, Capacitors_SMD:C_0402, symbol C
- removed IC1: ADS1299, Housings_QFP:TQFP-64_10x10mm_Pitch0.5mm, symbol ADS1299
- removed P3: CONN_01X08, symbol CONN_01X08
- removed R11, R12: 10k, Resistors_SMD:R_0402, symbol R
- removed R3, R4, R5: 30k, Resistors_SMD:R_0402, symbol R
- removed R6: 1MΩ, Resistors_SMD:R_0402, symbol R
- removed R7, R8: 100R, Resistors_SMD:R_0402, symbol R
- removed U4: MPU-9250, Housings_DFN_QFN:QFN-24_3x3mm_Pitch0.4mm, symbol MPU-9250
- removed U5, U6: INA828, INA828:SOIC_8_4.9mm_x_3.91, symbol INA128
Connections:
- net labels removed: BIASIN, IN1-, IN1N, IN1P, IN2-, IN2N, IN2P, IN3, IN34-, IN4, REF/SRB1, REF_ELECTRODE, SCL, SDI, VCAP1, VCAP2, VCAP3, VCAP4, VREFN, VREFP
- wire segments 353 -> 170
- no-connect marks 15 -> 0
Other:
- note removed: "C15 is tantalum"
- note removed: "CLKSEL should be = 1 (dig)"
- note removed: "Can use either 1.0nF or 1.5nF\n\nTODO: REDO SETUP (SEE GSK PAPER!)"
- note removed: "Caps: 1µF or 10µF"
- note removed: "Configuration for EEG and EMG different\nFor EEG, only channels 1-4 used\nUnused to AVDD"
- note removed: "If GPIO unused: Connect→10+kΩ→GND"
- note removed: "O1"
- note removed: "O2"
- note removed: "Oz"

Commit message: Linked new library (under libs_common). Added battery recharging circuit to schematic.
Parts:
- added C? (x2): 4.7uF, Capacitors_SMD:C_0402, symbol C
- added D?: LED, symbol LED
- added R?: 2k, symbol R
- added U?: MCP73831, symbol MCP73831
Connections:
- net labels added: 5V_in_charge
- wire segments 170 -> 194
- no-connect marks 0 -> 1
Other:
- note added: "Battery Connection"
Changed lines of the file:
@@
 LIBS:texas_TPS61222
 LIBS:EEG_ADS1299_2-cache
+LIBS:bioreactor
 LIBS:nrf52_sensor_array-cache
 EELAYER 25 0
@@
 	1    0    0    -1
 $EndComp
-$Comp
-L VCC #PWR02
-U 1 1 588ADF4F
-P 2450 6700
-F 0 "#PWR02" H 2450 6800 30  0001 C CNN
-F 1 "VCC" H 2450 6800 30  0000 C CNN
-F 2 "" H 2450 6700 60  0000 C CNN
-F 3 "" H 2450 6700 60  0000 C CNN
-	1    2450 6700
-	1    0    0    -1
-$EndComp
 Text Label 2700 7600 0    60   ~ 0
 SWDCLK
@@
 Text GLabel 11650 3850 2    60   Input ~ 0
 AVSS
-Text Label 2700 6800 0    60   ~ 0
+Text Label 8100 7350 0    60   ~ 0
 SYS_LOAD
 Text Label 9900 4450 0    60   ~ 0
@@
 Text Label 3300 3300 0    60   ~ 0
 Vout
+Text GLabel 7550 6050 0    60   Input ~ 0
+5V_in_charge
+$Comp
+L MCP73831 U?
+U 1 1 5B170649
+P 8750 6800
+F 0 "U?" H 8750 6900 60  0000 C CNN
+F 1 "MCP73831" H 8750 7150 60  0000 C CNN
+F 2 "" H 8750 6800 60  0001 C CNN
+F 3 "" H 8750 6800 60  0001 C CNN
+	1    8750 6800
+	1    0    0    -1
+$EndComp
+$Comp
+L C C?
+U 1 1 5B171CA0
+P 7500 6450
+F 0 "C?" H 7550 6550 40  0000 L CNN
+F 1 "4.7uF" H 7506 6365 40  0000 L CNN
+F 2 "Capacitors_SMD:C_0402" H 7538 6300 30  0001 C CNN
+F 3 "~" H 7500 6450 60  0000 C CNN
+	1    7500 6450
+	0    -1   -1   0
+$EndComp
 Wire Wire Line
 	22100 4800 20400 4800
@@
 	2950 3700 2950 4050
 Wire Wire Line
-	3150 3850 2700 3850
-Wire Wire Line
-	3150 3500 3150 3850
-Wire Wire Line
-	3650 3500 3150 3500
+	2700 3850 3150 3850
+Wire Wire Line
+	3150 3850 3150 3500
+Wire Wire Line
+	3150 3500 3650 3500
 Wire Wire Line
 	2950 3300 2950 3400
 Wire Wire Line
-	3650 3300 2950 3300
+	2950 3300 3650 3300
 Wire Wire Line
 	2700 3100 2850 3100
@@
 Connection ~ 5350 3300
 Wire Wire Line
-	5350 3550 5350 3300
+	5350 3300 5350 3550
 Connection ~ 4900 3300
 Wire Wire Line
@@
 Connection ~ 10800 4100
 Wire Wire Line
-	8600 4450 10800 4450
-Wire Wire Line
-	8600 4100 8600 4450
-Wire Wire Line
-	8800 4100 8600 4100
+	10800 4450 8600 4450
+Wire Wire Line
+	8600 4450 8600 4100
+Wire Wire Line
+	8600 4100 8800 4100
 Wire Wire Line
 	10800 4100 10500 4100
 Wire Wire Line
-	10800 4450 10800 3550
+	10800 3550 10800 4450
 Wire Wire Line
 	10800 3550 10500 3550
 Connection ~ 8350 3000
 Wire Wire Line
-	8350 2400 8350 3000
-Wire Wire Line
-	10700 2400 8350 2400
-Wire Wire Line
-	10700 3000 10700 2400
-Wire Wire Line
-	10500 3000 10700 3000
+	8350 3000 8350 2400
+Wire Wire Line
+	8350 2400 10700 2400
+Wire Wire Line
+	10700 2400 10700 3000
+Wire Wire Line
+	10700 3000 10500 3000
 Wire Wire Line
 	7450 3000 8800 3000
@@
 Wire Wire Line
 	2350 6800 2700 6800
-Wire Wire Line
-	2450 6800 2450 6700
 Wire Wire Line
 	2350 7000 2450 7000
@@
 Wire Wire Line
 	24400 6000 24700 6000
-Connection ~ 2450 6800
+Wire Wire Line
+	7700 6550 8250 6550
+Wire Wire Line
+	7800 6050 7800 6700
+Wire Wire Line
+	7800 6050 7550 6050
+Connection ~ 7800 6550
+Wire Wire Line
+	8250 6900 8100 6900
+Wire Wire Line
+	8100 6900 8100 7350
+Wire Wire Line
+	8100 7050 8250 7050
+Connection ~ 8100 7050
+Wire Wire Line
+	7350 6450 7300 6450
+Wire Wire Line
+	7300 6450 7300 6600
+Text GLabel 7300 6600 0    60   Input ~ 0
+DGND
+$Comp
+L LED D?
+U 1 1 5B1733AF
+P 10000 6450
+F 0 "D?" H 10000 6550 50  0000 C CNN
+F 1 "LED" H 10000 6350 50  0000 C CNN
+F 2 "" H 10000 6450 50  0001 C CNN
+F 3 "" H 10000 6450 50  0001 C CNN
+	1    10000 6450
+	0    -1   -1   0
+$EndComp
+Wire Wire Line
+	7800 6700 8250 6700
+Wire Wire Line
+	10000 6600 10000 7050
+Wire Wire Line
+	10000 7050 9250 7050
+Text GLabel 10000 6000 2    60   Input ~ 0
+DVDD
+Wire Wire Line
+	10000 6000 10000 6300
+Wire Wire Line
+	9250 6800 9550 6800
+Wire Wire Line
+	9450 6700 9450 6900
+Wire Wire Line
+	9450 6900 9250 6900
+Connection ~ 9450 6800
+Text GLabel 9550 6800 2    60   Input ~ 0
+DGND
+NoConn ~ 9250 6700
+Text Notes 8100 7450 0    60   ~ 0
+Battery Connection
+$Comp
+L C C?
+U 1 1 5B176C6B
+P 7850 7150
+F 0 "C?" H 7900 7250 40  0000 L CNN
+F 1 "4.7uF" H 7856 7065 40  0000 L CNN
+F 2 "Capacitors_SMD:C_0402" H 7888 7000 30  0001 C CNN
+F 3 "~" H 7850 7150 60  0000 C CNN
+	1    7850 7150
+	0    -1   -1   0
+$EndComp
+Text GLabel 7550 7150 0    60   Input ~ 0
+DGND
+Wire Wire Line
+	8100 7150 8000 7150
+Connection ~ 8100 7150
+Wire Wire Line
+	7700 7150 7550 7150
+Wire Wire Line
+	7700 6550 7700 6450
+Wire Wire Line
+	7700 6450 7650 6450
+$Comp
+L R R?
+U 1 1 5B177325
+P 9500 6550
+F 0 "R?" V 9580 6550 50  0000 C CNN
+F 1 "2k" V 9500 6550 50  0000 C CNN
+F 2 "" V 9430 6550 50  0001 C CNN
+F 3 "" H 9500 6550 50  0001 C CNN
+	1    9500 6550
+	0    1    1    0
+$EndComp
+Wire Wire Line
+	9350 6550 9250 6550
+Wire Wire Line
+	9650 6550 9750 6550
+Wire Wire Line
+	9750 6550 9750 6700
+Wire Wire Line
+	9750 6700 9450 6700
+Wire Wire Line
+	8100 7350 6850 7350
+Wire Wire Line
+	6850 7350 6850 7250
+$Comp
+L VCC #PWR?
+U 1 1 5B179102
+P 6850 7250
+F 0 "#PWR?" H 6850 7350 30  0001 C CNN
+F 1 "VCC" H 6850 7350 30  0000 C CNN
+F 2 "" H 6850 7250 60  0000 C CNN
+F 3 "" H 6850 7250 60  0000 C CNN
+	1    6850 7250
+	1    0    0    -1
+$EndComp
+Text GLabel 2700 6800 2    60   Input ~ 0
+5V_in_charge
 $EndSCHEMATC

Commit message: Added battery management (recharging, MCP73831) circuit to device, using 500 mA configuration.
Parts:
- added P3: CONN_2, Pin_Headers:Pin_Header_Straight_1x02_Pitch2.54mm, symbol CONN_2
- U4: renamed from U?; footprint (none) -> Housings_DFN_QFN:DFN-8-1EP_2x3mm_Pitch0.5mm
- gave numbers to parts that had none: 4
- renumbered C38 to C6, C39 to C7
Connections:
- wire segments 194 -> 196
Other:
- note added: "Battery Recharging Circuit"
- note added: "Load Switch Battery Measurement Controller"
- note removed: "Remove switch??"

Commit message: Updated schematic with all components. Plan is to replace multiplexers with ADG1606 (single supply), and get rid of -5V regulator.
Parts:
- removed D2: LED, LEDs:LED_0603, symbol LED-RESCUE-EEG_ADS1299_2
- added C10, C12, C14, C15, C16, C17, C18, C8, C9: 4.7uF, Capacitors_SMD:C_0402, symbol C
- added C11: 1uF, Capacitors_SMD:C_0402, symbol C
- added J1, J2, J3, J4, J5, J6: CONN_01X08, symbol CONN_01X08
- added MUX1, MUX2, MUX3: MUX36S16, symbol MUX36S16
- added R2, R3: 2k, symbol R
- added U5: LM27761, symbol LM27761
Connections:
- net labels added: -5VDD, LED1, SIG_OUT_D, Vin, ctr_m1_a0, ctr_m1_a1, ctr_m1_a2, ctr_m1_a3, ctr_m2_a0, ctr_m2_a1, ctr_m2_a2, ctr_m2_a3, ctr_m3_a0, ctr_m3_a1, ctr_m3_a2, ctr_m4_a3
- net labels removed: LED2, LED3
- wire segments 196 -> 398
- no-connect marks 1 -> 22
Other:
- note added: "5V Inverter"
- note added: "ALSO CONSIDER TYING THE CONTROLS TOGETHER, \nWE ARE MUXING AT ADC 3+1 INPUTS"
- note added: "CHANGE THESE MUXES TO ADG1606; No need for voltage inverter"
- note added: "LTC1046\nPDIP Packages?\n"
- note added: "NOT SURE WHAT THESE R VALUES SHOULD BE!"
- note added: "Sensor Array"
- note removed: "220Ω+"
- note removed: "Apparently supposed to be 3.3µH????\nSee TI forumns/ WEBENCH"
- note removed: "LEDV = 2.2V max."
- note removed: "LEDs [POWER; BLE; RDATAC]\nDo these need dropdown resistors??\nFor debugging only; will not be used in final version."
- note removed: "PWR LED"

Commit message: Removed old muxes and -5V reguator. Updated schematic and added ADG1606, and 2 rows of headers.
Parts:
- removed C10, C12, C14, C15, C16, C17, C18, C9: 4.7uF, Capacitors_SMD:C_0402, symbol C
- removed C11: 1uF, Capacitors_SMD:C_0402, symbol C
- removed J3, J4, J5, J6: CONN_01X08, symbol CONN_01X08
- removed MUX1, MUX2, MUX3: MUX36S16, symbol MUX36S16
- removed R2, R3: 2k, symbol R
- removed U5: LM27761, symbol LM27761
- added MUX1: ADG1606, Housings_DFN_QFN:QFN-32-1EP_5x5mm_Pitch0.5mm, symbol ADG1606
- J1, J2: footprint (none) -> Pin_Headers:Pin_Header_Straight_1x08_Pitch2.54mm
Connections:
- net labels added: m1_D_out
- net labels removed: -5VDD, SIG_OUT_D, ctr_m2_a0, ctr_m2_a1, ctr_m2_a2, ctr_m2_a3, ctr_m3_a0, ctr_m3_a1, ctr_m3_a2, ctr_m4_a3
- wire segments 398 -> 255
- no-connect marks 22 -> 8
Other:
- note removed: "5V Inverter"
- note removed: "LTC1046\nPDIP Packages?\n"
- note removed: "NOT SURE WHAT THESE R VALUES SHOULD BE!"

Commit message: Added ADC: ADS1220, added 2/3 Multiplexers (ADG1606)
Parts:
- added C10, C9: 0.1uF, Capacitors_SMD:C_0402, symbol C
- added C11, C12: 4.7uF, Capacitors_SMD:C_0402, symbol C
- added J3, J4, J5, J6: CONN_01X08, Pin_Headers:Pin_Header_Straight_1x08_Pitch2.54mm, symbol CONN_01X08
- added MUX2, MUX3: ADG1606, Housings_DFN_QFN:QFN-32-1EP_5x5mm_Pitch0.5mm, symbol ADG1606
- added U5: ADS1220, Housings_DFN_QFN:QFN-16-1EP_3x3mm_Pitch0.5mm, symbol ADS1220
Connections:
- net labels added: m2_D_out, m3_D_out, meas_REFERENCE
- net labels removed: ~PWDN/RESET
- wire segments 255 -> 348
- no-connect marks 8 -> 24
Other:
- note removed: "ALSO CONSIDER TYING THE CONTROLS TOGETHER, \nWE ARE MUXING AT ADC 3+1 INPUTS"
- note removed: "CHANGE THESE MUXES TO ADG1606; No need for voltage inverter"

Commit message: Updated .gitignore, added pins for 2 reference electrodes (grounded)
Parts:
- added P4: CONN_2, Pin_Headers:Pin_Header_Straight_1x02_Pitch2.54mm, symbol CONN_2
Connections:
- wire segments 348 -> 355
Changed lines of the file:
@@
 Wire Wire Line
 	12100 10850 12600 10850
+$Comp
+L CONN_2 P4
+U 1 1 5B1D9853
+P 14950 8800
+F 0 "P4" V 14900 8800 40  0000 C CNN
+F 1 "CONN_2" V 15000 8800 40  0000 C CNN
+F 2 "Pin_Headers:Pin_Header_Straight_1x02_Pitch2.54mm" H 14950 8800 60  0001 C CNN
+F 3 "" H 14950 8800 60  0000 C CNN
+	1    14950 8800
+	-1   0    0    -1
+$EndComp
+Text Label 16450 8650 0    60   ~ 0
+meas_REFERENCE
+Wire Wire Line
+	15300 8700 16450 8700
+Wire Wire Line
+	16450 8700 16450 8650
+Wire Wire Line
+	15300 8900 16450 8900
+Wire Wire Line
+	16450 8900 16450 8850
+Text Label 16450 8850 0    60   ~ 0
+meas_REFERENCE
+Wire Wire Line
+	16000 8700 16000 9150
+Wire Wire Line
+	16000 9150 16350 9150
+Connection ~ 16000 8700
+Wire Wire Line
+	16150 8900 16150 9150
+Connection ~ 16150 8900
+Connection ~ 16150 9150
+Text GLabel 16350 9150 2    60   Input ~ 0
+AVSS
 $EndSCHEMATC

Commit message: Added option to short Reference electrodes to ground (using pad N1).
Parts:
- added N1: N.C., Capacitors_SMD:C_0402, symbol C
Connections:
- wire segments 355 -> 356
Changed lines of the file:
@@
 Connection ~ 16150 8900
 Connection ~ 16150 9150
-Text GLabel 16350 9150 2    60   Input ~ 0
+$Comp
+L C N1
+U 1 1 5B1DC489
+P 16500 9150
+F 0 "N1" H 16550 9250 40  0000 L CNN
+F 1 "N.C." H 16506 9065 40  0000 L CNN
+F 2 "Capacitors_SMD:C_0402" H 16538 9000 30  0001 C CNN
+F 3 "~" H 16500 9150 60  0000 C CNN
+	1    16500 9150
+	0    -1   -1   0
+$EndComp
+Wire Wire Line
+	16650 9150 16850 9150
+Text GLabel 16850 9150 2    60   Input ~ 0
 AVSS
 $EndSCHEMATC
