File: nrf52_sensor_array.sch (KiCad schematic (older format))
At the start: 60 parts, among them J1 CONN_01X08, J2 CONN_01X08, J3 CONN_01X08, J4 CONN_01X08, J5 CONN_01X08, J6 CONN_01X08, P1 CONN_2, P2 CONN_2, P3 CONN_2, P4 CONN_2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

Commit message: Added voltage divider, pins for 3v3 power supply.
Parts:
- removed N1: N.C., Capacitors_SMD:C_0402, symbol C
- added P5: CONN_2, Pin_Headers:Pin_Header_Straight_1x02_Pitch2.54mm, symbol CONN_2
- added R2: 2k, symbol R
Connections:
- wire segments 356 -> 359
Other:
- note added: "From Temp sensors"
- note added: "Voltage divider"
